Commit message: FEAT: Multi-Modal General Purpose Suite. Thermal/Acoustic sensing, Mission State Machine, and Dynamic Holographic Shaders.

File: vectorsense_ws/src/vectorsense_description/urdf/drone_high_fidelity.urdf (robot description, URDF)
Before this commit: robot vectorsense_drone, 6 links, 5 joints
Links:
- removed link motor_fl_link
- removed link motor_fr_link
- added link acoustic_sensor_link; visual sphere radius=0.03
- added link thermal_camera_link; visual box size=0.05 0.05 0.05
Joints:
- removed joint motor_fl_joint
- removed joint motor_fr_joint
- added joint acoustic_joint: type fixed, parent base_link, child acoustic_sensor_link, origin xyz=-0.1 0 0 rpy=0 0 0
- added joint thermal_joint: type fixed, parent base_link, child thermal_camera_link, origin xyz=0.1 0 0 rpy=0 0 0
