Commit message: Defense-Grade Prototype Overhaul: Ghost Core URDF, Sub-10ms LZ4/ZMQ Bridge, Full-Bleed Glassmorphism UI, and Autonomous Flight State Machine.

File: vectorsense_ws/src/vectorsense_megacomplex/urdf/vectorsense_ghost.urdf.xacro (robot description, xacro)
@@ -1,6 +1,7 @@
 <?xml version="1.0"?>
 <robot xmlns:xacro="http://www.ros.org/wiki/xacro" name="vectorsense_drone">
-  <!-- Stable Ghost Core Inertial -->
+  <!-- THE GHOST CORE: Mathematically Perfect Physics Skeleton -->
   <link name="base_link">
+    <!-- PHYSICS CORE: Zero-Visual, Perfectly Symmetric Intertials -->
     <inertial>
       <origin xyz="0 0 0" rpy="0 0 0"/>
@@ -8,37 +9,40 @@
       <inertia ixx="0.03" ixy="0" ixz="0" iyy="0.03" iyz="0" izz="0.06"/>
     </inertial>
+    <!-- COLLISION CORE: Primitive-only to prevent mesh shears -->
     <collision name="base_collision">
+      <origin xyz="0 0 0" rpy="0 0 0"/>
       <geometry>
         <box size="0.2 0.2 0.1"/>
       </geometry>
     </collision>
-    <!-- Visual Skin: Dressing the ghost -->
-    <visual>
+    <!-- VISUAL SKINS: Weightless CAD layers (No Collision / No Inertial) -->
+    <visual name="skin_base">
       <geometry>
         <mesh filename="package://vectorsense_megacomplex/meshes/DroneFYDPBase.stl" scale="0.001 0.001 0.001"/>
       </geometry>
     </visual>
+    <visual name="skin_xbeam">
+      <origin xyz="0 0 0.05" rpy="0 0 0"/>
+      <geometry>
+        <mesh filename="package://vectorsense_megacomplex/meshes/Xbeam.stl" scale="0.001 0.001 0.001"/>
+      </geometry>
+    </visual>
+    <visual name="skin_beam180">
+      <origin xyz="0 0 0.05" rpy="0 0 1.5708"/>
+      <geometry>
+        <mesh filename="package://vectorsense_megacomplex/meshes/180beam.stl" scale="0.001 0.001 0.001"/>
+      </geometry>
+    </visual>
+    <visual name="skin_top_plate">
+      <origin xyz="0 0 0.1" rpy="0 0 0"/>
+      <geometry>
+        <mesh filename="package://vectorsense_megacomplex/meshes/top_plate.stl" scale="0.001 0.001 0.001"/>
+      </geometry>
+    </visual>
   </link>
-  <!-- Weightless Visual Attachments -->
-  <xacro:macro name="visual_part" params="name mesh_file x y z yaw">
-    <link name="${name}_link">
-      <visual>
-        <geometry>
-          <mesh filename="package://vectorsense_megacomplex/meshes/${mesh_file}" scale="0.001 0.001 0.001"/>
-        </geometry>
-      </visual>
-    </link>
-    <joint name="${name}_joint" type="fixed">
-      <parent link="base_link"/>
-      <child link="${name}_link"/>
-      <origin xyz="${x} ${y} ${z}" rpy="0 0 ${yaw}"/>
-    </joint>
-  </xacro:macro>
-  <xacro:visual_part name="xbeam" mesh_file="Xbeam.stl" x="0" y="0" z="0.05" yaw="0"/>
-  <xacro:visual_part name="beam180" mesh_file="180beam.stl" x="0" y="0" z="0.05" yaw="1.5708"/>
-  <xacro:visual_part name="top_plate" mesh_file="top_plate.stl" x="0" y="0" z="0.1" yaw="0"/>
-  <!-- Motors and Propulsion -->
+  <!-- MOTORS: Exact Symmetry (X,Y = +/- 0.225m) -->
   <xacro:macro name="motor" params="name x y index direction">
     <link name="motor_${name}">
+      <!-- Weightless visual anchor -->
       <visual>
         <geometry>
@@ -46,4 +50,9 @@
         </geometry>
       </visual>
+      <!-- Small placeholder inertial to satisfy some solvers, though visual-only is intended -->
+      <inertial>
+        <mass value="0.001"/>
+        <inertia ixx="0.0001" ixy="0" ixz="0" iyy="0.0001" iyz="0" izz="0.0001"/>
+      </inertial>
     </link>
     <joint name="motor_${name}_joint" type="continuous">
@@ -72,8 +81,8 @@
     </gazebo>
   </xacro:macro>
-  <xacro:motor name="fr" x="0.25" y="-0.25" index="0" direction="ccw"/>
-  <xacro:motor name="fl" x="0.25" y="0.25" index="1" direction="cw"/>
-  <xacro:motor name="br" x="-0.25" y="-0.25" index="2" direction="cw"/>
-  <xacro:motor name="bl" x="-0.25" y="0.25" index="3" direction="ccw"/>
+  <xacro:motor name="fr" x="0.225" y="-0.225" index="0" direction="ccw"/>
+  <xacro:motor name="fl" x="0.225" y="0.225" index="1" direction="cw"/>
+  <xacro:motor name="br" x="-0.225" y="-0.225" index="2" direction="cw"/>
+  <xacro:motor name="bl" x="-0.225" y="0.225" index="3" direction="ccw"/>
   <gazebo>
     <plugin filename="gz-sim-multicopter-velocity-control-system" name="gz::sim::systems::MulticopterVelocityControl">
@@ -85,4 +94,8 @@
       <maximumAngularVelocity>5.0</maximumAngularVelocity>
     </plugin>
+    <!-- State Publisher for Odometry -->
+    <plugin filename="gz-sim-odometry-publisher-system" name="gz::sim::systems::OdometryPublisher">
+      <dimensions>3</dimensions>
+    </plugin>
   </gazebo>
 </robot>

Commit message: feat: professional Apple-grade dashboard with full demo capability
- Complete monochrome design system (App.css) - zero emojis, Apple-inspired glassmorphism
- SpatialTwin: full hexacopter 3D model with 6 animated rotors, mode-driven scan cone colours, industrial facility (tanks + distillation tower + pipes), gas leak haze animation
- Manual flight: WASD + F (alt up) / C (alt down) keyboard controls wired to local state + WS bridge
- On-screen flight pad repositioned to bottom-centre, no longer overlapping SCADA or advisory panels
- MissionControl: 4 active-protocol modes with black-fill active state, live advisory banner
- MitigationControl: two-tap confirmation flow, all 4 SCADA commands visible, scrollable sidebar
- DroneSpecs: tabbed technical spec table (Airframe/Propulsion/Sensors/Intelligence) + Why-Best cards
- ThreatEconomics: PINN-derived gas classification (VOC/CH4/H2S/CO), regulatory exposure USD/hr, confidence scoring from NS residual, event timeline
- SystemDiagnostics: infrastructure status grid (ZMQ/PINN/DCS/ROS2), PINN kernel metrics, live system log
- financial_physics_bridge.py: WASD manual override support
- Git LFS configured for *.mp4 *.mov *.avi *.mkv
- demo video.mp4 tracked via Git LFS (1.1 GB)

File: vectorsense_ws/src/vectorsense_megacomplex/urdf/vectorsense_ghost.urdf.xacro (robot description, xacro)
@@ -41,8 +41,7 @@
     </visual>
   </link>
-  <!-- MOTORS: Exact Symmetry (X,Y = +/- 0.225m) -->
+  <!-- MOTORS: Exact Symmetry (Hexacopter configuration) -->
   <xacro:macro name="motor" params="name x y index direction">
     <link name="motor_${name}">
-      <!-- Weightless visual anchor -->
       <visual>
         <geometry>
@@ -50,5 +49,4 @@
         </geometry>
       </visual>
-      <!-- Small placeholder inertial to satisfy some solvers, though visual-only is intended -->
       <inertial>
         <mass value="0.001"/>
@@ -71,5 +69,5 @@
         <timeConstantDown>0.025</timeConstantDown>
         <maxRotVelocity>1500</maxRotVelocity>
-        <motorConstant>8.54858e-06</motorConstant>
+        <motorConstant>8.54858e-04</motorConstant>
         <momentConstant>0.016</momentConstant>
         <commandSubTopic>command/motor_speed</commandSubTopic>
@@ -81,8 +79,43 @@
     </gazebo>
   </xacro:macro>
-  <xacro:motor name="fr" x="0.225" y="-0.225" index="0" direction="ccw"/>
-  <xacro:motor name="fl" x="0.225" y="0.225" index="1" direction="cw"/>
-  <xacro:motor name="br" x="-0.225" y="-0.225" index="2" direction="cw"/>
-  <xacro:motor name="bl" x="-0.225" y="0.225" index="3" direction="ccw"/>
+  <!-- Hexacopter Arms (60 deg separation) -->
+  <xacro:motor name="front_right" x="0.3" y="-0.17" index="0" direction="ccw"/>
+  <xacro:motor name="right" x="0" y="-0.34" index="1" direction="cw"/>
+  <xacro:motor name="back_right" x="-0.3" y="-0.17" index="2" direction="ccw"/>
+  <xacro:motor name="back_left" x="-0.3" y="0.17" index="3" direction="cw"/>
+  <xacro:motor name="left" x="0" y="0.34" index="4" direction="ccw"/>
+  <xacro:motor name="front_left" x="0.3" y="0.17" index="5" direction="cw"/>
+  <!-- SENSING PAYLOAD -->
+  <link name="lidar_link">
+    <visual>
+      <geometry><cylinder radius="0.05" length="0.05"/></geometry>
+      <material name="black"><color rgba="0 0 0 1"/></material>
+    </visual>
+  </link>
+  <joint name="lidar_joint" type="fixed">
+    <parent link="base_link"/>
+    <child link="lidar_link"/>
+    <origin xyz="0 0 0.15" rpy="0 0 0"/>
+  </joint>
+  <gazebo reference="lidar_link">
+    <sensor name="gpu_lidar" type="gpu_lidar">
+      <update_rate>10</update_rate>
+      <lidar>
+        <scan>
+          <horizontal>
+            <samples>360</samples>
+            <resolution>1</resolution>
+            <min_angle>-3.14159</min_angle>
+            <max_angle>3.14159</max_angle>
+          </horizontal>
+        </scan>
+        <range>
+          <min>0.2</min>
+          <max>30.0</max>
+        </range>
+      </lidar>
+      <gz_frame_id>lidar_link</gz_frame_id>
+    </sensor>
+  </gazebo>
   <gazebo>
     <plugin filename="gz-sim-multicopter-velocity-control-system" name="gz::sim::systems::MulticopterVelocityControl">
@@ -94,8 +127,9 @@
       <maximumAngularVelocity>5.0</maximumAngularVelocity>
     </plugin>
-    <!-- State Publisher for Odometry -->
     <plugin filename="gz-sim-odometry-publisher-system" name="gz::sim::systems::OdometryPublisher">
       <dimensions>3</dimensions>
     </plugin>
+    <plugin filename="gz-sim-imu-system" name="gz::sim::systems::Imu">
+    </plugin>
   </gazebo>
 </robot>
